Commit message: change camera xacro

File: src/dogbot/urdf/camera.xacro (robot description, xacro)
@@ -1,5 +1,5 @@
 <?xml version="1.0"?>
 <robot xmlns:xacro="http://www.ros.org/wiki/xacro" name="camera">
-    <xacro:macro name="usb_camera" params="prefix:=camera">
+    <xacro:macro name="camera_link" params="prefix:=camera">
         <!-- Create laser reference frame -->
         <link name="${prefix}_link">

Commit message: change camera xacro

File: src/dogbot/urdf/camera.xacro (robot description, xacro)
@@ -1,5 +1,5 @@
 <?xml version="1.0"?>
 <robot xmlns:xacro="http://www.ros.org/wiki/xacro" name="camera">
-    <xacro:macro name="camera_link" params="prefix:=camera">
+    <xacro:macro name="web_camera" params="prefix:=camera">
         <!-- Create laser reference frame -->
         <link name="${prefix}_link">

Commit message: change camera xacro

File: src/dogbot/urdf/camera.xacro (robot description, xacro)
@@ -3,24 +3,24 @@
     <xacro:macro name="web_camera" params="prefix:=camera">
         <!-- Create laser reference frame -->
-        <link name="${prefix}_link">
-            <inertial>
-                <origin rpy="0 0 0" xyz="0.1 0 0.15"/>
-                <mass value="0.01" />
-                <inertia ixx="0.4" ixy="0.0" ixz="0.0" iyy="0.4" iyz="0.0" izz="0.4" />
-            </inertial>
-            <visual>
-                <material name = "white_1"/>
-                <origin rpy="0 0 0" xyz="0.1 0 0.15"/>
-                <geometry>
-                    <box size="0.3 0.3 0.1" />
-                </geometry>
-             </visual>
-            <collision>
-                <origin rpy="0 0 0" xyz="0.1 0 0.15"/>
-                <geometry>
-                    <box size="0.3 0.3 0.1" />
-                </geometry>
-            </collision>
-        </link>
+        <link name = "camera_link">
+   <visual>
+     <material name = "white_1"/>
+     <origin rpy="0 0 0" xyz="0.1 0 0.15"/>
+    <geometry>
+     <box size="0.3 0.3 0.1" />
+    </geometry>
+    </visual>
+    <collision>
+     <origin rpy="0 0 0" xyz="0.1 0 0.15"/>
+    <geometry>
+     <box size="0.3 0.3 0.1" />
+    </geometry>
+    </collision>
+    <inertial>
+     <origin rpy="0 0 0" xyz="0.1 0 0.15"/>
+      <mass value="0.01" />
+      <inertia ixx="0.4" ixy="0.0" ixz="0.0" iyy="0.4" iyz="0.0" izz="0.4" />
+  </inertial>
+   </link>
         <gazebo reference="${prefix}_link">
             <material>Gazebo/Black</material>
