Commit message: change camera_link

File: src/dogbot/urdf/camera_1.xacro (robot description, xacro)
@@ -32,6 +32,6 @@
                     <horizontal_fov>1.3962634</horizontal_fov>
                     <image>
-                        <width>1280</width>
-                        <height>720</height>
+                        <width>320</width>
+                        <height>180</height>
                         <format>R8G8B8</format>
                     </image>

File: src/dogbot/urdf/dogbot.urdf (robot description, URDF)
Before this commit: robot dogbot, 10 links, 9 joints
Links:
- removed link back_leg_left
- removed link back_leg_left2
- removed link back_leg_right
- removed link back_leg_right2
- removed link base_link
- removed link camera_link
- removed link front_leg_left
- removed link front_leg_left2
- removed link front_leg_right
- removed link front_leg_right2
Joints:
- removed joint camera_joint
- removed joint joint_b_l_1
- removed joint joint_b_l_2
- removed joint joint_b_r_1
- removed joint joint_b_r_2
- removed joint joint_f_l_1
- removed joint joint_f_l_2
- removed joint joint_f_r_1
- removed joint joint_f_r_2
