Commit message: add camera

File: src/dogbot/urdf/dogbot.urdf (robot description, URDF)
Before this commit: robot dogbot, 10 links, 8 joints
Joints:
- added joint camera_joint: type fixed, parent base_link, child camera_link, origin xyz=0.5 0 0.6

Commit message: adjust camera pos

File: src/dogbot/urdf/dogbot.urdf (robot description, URDF)
Before this commit: robot dogbot, 10 links, 9 joints
Joints:
- joint camera_joint: origin xyz=0.5 0 0.6 -> xyz=0.45 0 0.6

Commit message: adjust camera pos

File: src/dogbot/urdf/dogbot.urdf (robot description, URDF)
Before this commit: robot dogbot, 10 links, 9 joints
Links:
- link camera_link: geometry collision box size=0.3 0.3 0.1; visual box size=0.3 0.3 0.1

Commit message: adjust camera pos

File: src/dogbot/urdf/dogbot.urdf (robot description, URDF)
Before this commit: robot dogbot, 10 links, 9 joints
Joints:
- joint camera_joint: origin xyz=0.45 0 0.6 -> xyz=0 0 0.6

Commit message: adjust camera pos

File: src/dogbot/urdf/dogbot.urdf (robot description, URDF)
Before this commit: robot dogbot, 10 links, 9 joints
Joints:
- joint camera_joint: origin xyz=0 0 0.6 -> xyz=0 0 0

Commit message: adjust camera pos

File: src/dogbot/urdf/dogbot.urdf (robot description, URDF)
Before this commit: robot dogbot, 10 links, 9 joints
Joints:
- joint camera_joint: origin xyz=0 0 0 -> xyz=0 0 0.1

Commit message: adjust camera pos

File: src/dogbot/urdf/dogbot.urdf (robot description, URDF)
Before this commit: robot dogbot, 10 links, 9 joints
Joints:
- joint camera_joint: origin xyz=0 0 0.1 -> xyz=0 0 -0.1

Commit message: adjust camera pos

File: src/dogbot/urdf/dogbot.urdf (robot description, URDF)
Before this commit: robot dogbot, 10 links, 9 joints
Joints:
- joint camera_joint: origin xyz=0 0 -0.1 -> xyz=0 0 0.2

Commit message: adjust camera pos

File: src/dogbot/urdf/dogbot.urdf (robot description, URDF)
Before this commit: robot dogbot, 10 links, 9 joints
Links:
- link base_link: geometry collision box size=1 0.3 0.2; visual box size=1 0.3 0.2
Joints:
- joint camera_joint: origin xyz=0 0 0.2 -> xyz=0 0 0.6

Commit message: adjust camera pos

File: src/dogbot/urdf/dogbot.urdf (robot description, URDF)
Before this commit: robot dogbot, 10 links, 9 joints
Joints:
- joint camera_joint: origin xyz=0 0 0.6 -> xyz=0 0 0.2

Commit message: adjust camera pos

File: src/dogbot/urdf/dogbot.urdf (robot description, URDF)
Before this commit: robot dogbot, 10 links, 9 joints
Joints:
- joint camera_joint: origin xyz=0 0 0.2 -> xyz=0.5 0 0.2

Commit message: adjust camera pos

File: src/dogbot/urdf/dogbot.urdf (robot description, URDF)
Before this commit: robot dogbot, 10 links, 9 joints
Joints:
- joint camera_joint: origin xyz=0.5 0 0.2 -> xyz=0.5 0 0.19

Commit message: adjust camera pos

File: src/dogbot/urdf/dogbot.urdf (robot description, URDF)
Before this commit: robot dogbot, 10 links, 9 joints
Joints:
- joint camera_joint: origin xyz=0.5 0 0.19 -> xyz=0.1 0 0.19

Commit message: change camera xacro

File: src/dogbot/urdf/dogbot.urdf (robot description, URDF)
Before this commit: robot dogbot, 9 links, 9 joints
Joints:
- joint camera_joint: origin xyz=0.1 0 0.19 -> xyz=0.1 0 0.19 rpy=0 0 0

Commit message: change camera xacro

File: src/dogbot/urdf/dogbot.urdf (robot description, URDF)
Before this commit: robot dogbot, 9 links, 9 joints
Links:
- added link camera_link, mass 0.01; collision box size=0.3 0.3 0.1; visual box size=0.3 0.3 0.1
Joints:
- joint camera_joint: origin xyz=0.1 0 0.19 rpy=0 0 0 -> xyz=0.1 0 0.19

Commit message: change camera gazebo

File: src/dogbot/urdf/dogbot.urdf (robot description, URDF)
Before this commit: robot dogbot, 10 links, 9 joints
Links:
- removed link camera_link

Commit message: change camera gazebo

File: src/dogbot/urdf/dogbot.urdf (robot description, URDF)
Before this commit: robot dogbot, 9 links, 9 joints
Links:
- added link camera_link, mass 0.01; collision box size=0.3 0.3 0.1; visual box size=0.3 0.3 0.1

Commit message: change camera_link

File: src/dogbot/urdf/dogbot.urdf (robot description, URDF)
Before this commit: robot dogbot, 0 links, 0 joints
Links:
- added link back_leg_left, mass 0.03; collision box size=0.1 0.1 0.3; visual box size=0.1 0.1 0.3
- added link back_leg_left2, mass 0.03; collision box size=0.07 0.07 0.4; visual box size=0.07 0.07 0.4
- added link back_leg_right, mass 0.03; collision box size=0.1 0.1 0.3; visual box size=0.1 0.1 0.3
- added link back_leg_right2, mass 0.03; collision box size=0.07 0.07 0.4; visual box size=0.07 0.07 0.4
- added link base_link, mass 0.03; collision box size=1 0.3 0.2; visual box size=1 0.3 0.2
- added link camera_link, mass 0.01; collision box size=0.3 0.3 0.1; visual box size=0.3 0.3 0.1
- added link front_leg_left, mass 0.03; collision box size=0.1 0.1 0.3; visual box size=0.1 0.1 0.3
- added link front_leg_left2, mass 0.03; collision box size=0.07 0.07 0.4; visual box size=0.07 0.07 0.4
- added link front_leg_right, mass 0.03; collision box size=0.1 0.1 0.3; visual box size=0.1 0.1 0.3
- added link front_leg_right2, mass 0.03; collision box size=0.07 0.07 0.4; visual box size=0.07 0.07 0.4
Joints:
- added joint camera_joint: type fixed, parent base_link, child camera_link, origin xyz=0.1 0 0.19
- added joint joint_b_l_1: type revolute, parent base_link, child back_leg_left, origin xyz=-0.2 -0.2 0.5, axis 0 1 0, limit lower=-1 upper=1 effort=4 velocity=2
- added joint joint_b_l_2: type revolute, parent back_leg_left, child back_leg_left2, origin xyz=0 0 -0.3, axis 0 1 0, limit lower=-2 upper=0 effort=4 velocity=2
- added joint joint_b_r_1: type revolute, parent base_link, child back_leg_right, origin xyz=-0.2 0.2 0.5, axis 0 1 0, limit lower=-1 upper=1 effort=4 velocity=2
- added joint joint_b_r_2: type revolute, parent back_leg_right, child back_leg_right2, origin xyz=0 0 -0.3, axis 0 1 0, limit lower=-2 upper=0 effort=4 velocity=2
- added joint joint_f_l_1: type revolute, parent base_link, child front_leg_left, origin xyz=0.2 -0.2 0.5 rpy=0 0 0 , axis 0 1 0, limit lower=-1 upper=1 effort=4 velocity=2
- added joint joint_f_l_2: type revolute, parent front_leg_left, child front_leg_left2, origin xyz=0 0 -0.3, axis 0 1 0, limit lower=-2 upper=0 effort=4 velocity=2
- added joint joint_f_r_1: type revolute, parent base_link, child front_leg_right, origin xyz=0.2 0.2 0.5, axis 0 1 0, limit lower=-1 upper=1 effort=4 velocity=2
- added joint joint_f_r_2: type revolute, parent front_leg_right, child front_leg_right2, origin xyz=0 0 -0.3, axis 0 1 0, limit lower=-2 upper=0 effort=4 velocity=2
